File: sdcard.brd (EAGLE design)
At the start: 31.9 x 36.1 mm, 6 parts, among them IC1 TLV75533PDRVR, IC2 TXB0108PWR, J1 2201778-1

Commit message: Add files via upload
Other:
- board size 31.9 x 36.1 mm -> 25.2 x 36.1 mm
- board text added: "Max Wolf 2019 Level Shifting SD Breakout V1"
- board text removed: "Max Wolf 2018 Level Shifting SD Breakout V1"
Changed lines of the file:
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@@
 <board>
 <plain>
-<wire x1="0.2" y1="0" x2="32.1" y2="0" width="0" layer="20"/>
-<wire x1="32.1" y1="0" x2="32.1" y2="36.1" width="0" layer="20"/>
-<wire x1="32.1" y1="36.1" x2="0.2" y2="36.1" width="0" layer="20"/>
+<wire x1="0.2" y1="0" x2="25.4" y2="0" width="0" layer="20"/>
+<wire x1="25.4" y1="0" x2="25.4" y2="36.1" width="0" layer="20"/>
+<wire x1="25.4" y1="36.1" x2="0.2" y2="36.1" width="0" layer="20"/>
 <wire x1="0.2" y1="36.1" x2="0.2" y2="0" width="0" layer="20"/>
-<text x="30.5" y="1" size="1.778" layer="1" rot="R90">Max Wolf 2018
+<dimension x1="0.2" y1="0" x2="0.2" y2="36.1" x3="-6.5" y3="18.05" textsize="1.778" layer="1"/>
+<text x="21" y="20.2" size="0.5" layer="1" rot="R90">Max Wolf 2019
 Level Shifting SD Breakout V1</text>
-<dimension x1="0.2" y1="0" x2="0.2" y2="36.1" x3="-6.5" y3="18.05" textsize="1.778" layer="1"/>
-<dimension x1="0.2" y1="0" x2="32.1" y2="0" x3="16.15" y3="-3.9" textsize="1.778" layer="1"/>
+<dimension x1="0.2" y1="0" x2="25.4" y2="0" x3="12.8" y3="-2" textsize="0.5" layer="1"/>
 </plain>
 <attributes>
@@
 <vertex x="0.2" y="36.1"/>
 <vertex x="0.2" y="0"/>
-<vertex x="32.1" y="0"/>
-<vertex x="32.1" y="36.1"/>
+<vertex x="25.4" y="0"/>
+<vertex x="25.4" y="36.1"/>
 </polygon>
 </signal>
